Commit message: colors actually do work, links were all just set to gray

File: nuturtle_description/urdf/turtlebot3_burger.urdf.xacro (robot description, xacro)
@@ -2,5 +2,5 @@
 <robot name="turtlebot3_burger"
   xmlns:xacro="http://ros.org/wiki/xacro">
-  <xacro:include filename="$(find nuturtle_description)/urdf/common_properties.urdf"/>
+  <xacro:include filename="$(find nuturtle_description)/urdf/common_properties.urdf.xacro"/>
   <link name="base_footprint"/>
   <joint name="base_joint" type="fixed">
@@ -41,5 +41,5 @@
         <mesh filename="package://nuturtle_description/meshes/left_tire.stl" scale="0.001 0.001 0.001"/>
       </geometry>
-      <material name="dark"/>
+      <material name="black"/>
     </visual>
     <collision>
@@ -67,5 +67,5 @@
         <mesh filename="package://nuturtle_description/meshes/right_tire.stl" scale="0.001 0.001 0.001"/>
       </geometry>
-      <material name="dark"/>
+      <material name="black"/>
     </visual>
     <collision>
@@ -116,5 +116,5 @@
         <mesh filename="package://nuturtle_description/meshes/lds.stl" scale="0.001 0.001 0.001"/>
       </geometry>
-      <material name="dark"/>
+      <material name="brown"/>
     </visual>
     <collision>

Commit message: add diff_params.yaml and begin integrating it into xacro files

File: nuturtle_description/urdf/turtlebot3_burger.urdf.xacro (robot description, xacro)
@@ -1,6 +1,11 @@
 <?xml version="1.0" ?>
-<robot name="turtlebot3_burger"
+<robot name="nuturtle_burger"
   xmlns:xacro="http://ros.org/wiki/xacro">
   <xacro:include filename="$(find nuturtle_description)/urdf/common_properties.urdf.xacro"/>
+  <xacro:property name="config_file" value="$(find nuturtle_description)/config/diff_params.yaml" />
+  <xacro:property name="params" value="${xacro.load_yaml(config_file)}"/>
+  <xacro:property name="wheel_radius" value="${params['/**']['ros__parameters']['wheel_radius']}"/>
+  <xacro:property name="track_width" value="${params['/**']['ros__parameters']['track_width']}"/>
+  <xacro:property name="collision_radius" value="${params['/**']['ros__parameters']['wheel_radius']}"/>
   <link name="base_footprint"/>
   <joint name="base_joint" type="fixed">
@@ -20,5 +25,6 @@
       <origin xyz="-0.032 0 0.070" rpy="0 0 0"/>
       <geometry>
-        <box size="0.140 0.140 0.143"/>
+        <cylinder radius="${collision_radius}" length="0.143"/>
+        <!-- <box size="0.140 0.140 0.143"/> -->
       </geometry>
     </collision>
@@ -32,5 +38,5 @@
     <parent link="base_link"/>
     <child link="wheel_left_link"/>
-    <origin xyz="0.0 0.08 0.023" rpy="-1.57 0 0"/>
+    <origin xyz="0.0 ${track_width/2} 0.023" rpy="-1.57 0 0"/>
     <axis xyz="0 0 1"/>
   </joint>
@@ -46,5 +52,5 @@
       <origin xyz="0 0 0" rpy="0 0 0"/>
       <geometry>
-        <cylinder length="0.018" radius="0.033"/>
+        <cylinder length="0.018" radius="${wheel_radius}"/>
       </geometry>
     </collision>
@@ -58,5 +64,5 @@
     <parent link="base_link"/>
     <child link="wheel_right_link"/>
-    <origin xyz="0.0 -0.080 0.023" rpy="-1.57 0 0"/>
+    <origin xyz="0.0 -${track_width/2} 0.023" rpy="-1.57 0 0"/>
     <axis xyz="0 0 1"/>
   </joint>
@@ -72,5 +78,5 @@
       <origin xyz="0 0 0" rpy="0 0 0"/>
       <geometry>
-        <cylinder length="0.018" radius="0.033"/>
+        <cylinder length="0.018" radius="${wheel_radius}"/>
       </geometry>
     </collision>

Commit message: add if condition to urdf so to handle positive vs negative collision_radius

File: nuturtle_description/urdf/turtlebot3_burger.urdf.xacro (robot description, xacro)
@@ -7,5 +7,5 @@
   <xacro:property name="wheel_radius" value="${params['/**']['ros__parameters']['wheel_radius']}"/>
   <xacro:property name="track_width" value="${params['/**']['ros__parameters']['track_width']}"/>
-  <xacro:property name="collision_radius" value="${params['/**']['ros__parameters']['wheel_radius']}"/>
+  <xacro:property name="collision_radius" value="${params['/**']['ros__parameters']['collision_radius']}"/>
   <link name="base_footprint"/>
   <joint name="base_joint" type="fixed">
@@ -25,6 +25,10 @@
       <origin xyz="-0.032 0 0.070" rpy="0 0 0"/>
       <geometry>
-        <cylinder radius="${collision_radius}" length="0.143"/>
-        <!-- <box size="0.140 0.140 0.143"/> -->
+        <xacro:if value="${collision_radius &lt; 0}">
+          <box size="0.140 0.140 0.143"/>
+        </xacro:if>
+        <xacro:if value="${collision_radius &gt; 0}">
+          <cylinder radius="${collision_radius}" length="0.143"/>
+        </xacro:if>
       </geometry>
     </collision>

Commit message: color argument added to urdf. Created utils.xacro to define colors and later on macros if I need them

File: nuturtle_description/urdf/turtlebot3_burger.urdf.xacro (robot description, xacro)
@@ -2,5 +2,6 @@
 <robot name="nuturtle_burger"
   xmlns:xacro="http://ros.org/wiki/xacro">
-  <xacro:include filename="$(find nuturtle_description)/urdf/common_properties.urdf.xacro"/>
+  <xacro:arg name="color" default="purple"/>
+  <xacro:include filename="$(find nuturtle_description)/urdf/utils.xacro"/>
   <xacro:property name="config_file" value="$(find nuturtle_description)/config/diff_params.yaml" />
   <xacro:property name="params" value="${xacro.load_yaml(config_file)}"/>
@@ -20,5 +21,5 @@
         <mesh filename="package://nuturtle_description/meshes/burger_base.stl" scale="0.001 0.001 0.001"/>
       </geometry>
-      <material name="light_black"/>
+      <material name="$(arg color)"/>
     </visual>
     <collision>
@@ -51,5 +52,5 @@
         <mesh filename="package://nuturtle_description/meshes/left_tire.stl" scale="0.001 0.001 0.001"/>
       </geometry>
-      <material name="black"/>
+      <material name="light_black"/>
     </visual>
     <collision>
@@ -77,5 +78,5 @@
         <mesh filename="package://nuturtle_description/meshes/right_tire.stl" scale="0.001 0.001 0.001"/>
       </geometry>
-      <material name="black"/>
+      <material name="light_black"/>
     </visual>
     <collision>
@@ -126,5 +127,5 @@
         <mesh filename="package://nuturtle_description/meshes/lds.stl" scale="0.001 0.001 0.001"/>
       </geometry>
-      <material name="brown"/>
+      <material name="light_black"/>
     </visual>
     <collision>

Commit message: nuturtle_description passed colcon test

File: nuturtle_description/urdf/turtlebot3_burger.urdf.xacro (robot description, xacro)
@@ -1,61 +1,65 @@
-<?xml version="1.0" ?>
+<?xml version="1.0"?>
 <robot name="nuturtle_burger"
   xmlns:xacro="http://ros.org/wiki/xacro">
-  <xacro:arg name="color" default="purple"/>
-  <xacro:include filename="$(find nuturtle_description)/urdf/utils.xacro"/>
+  <xacro:arg name="color" default="purple" />
+  <xacro:include filename="$(find nuturtle_description)/urdf/utils.xacro" />
   <xacro:property name="config_file" value="$(find nuturtle_description)/config/diff_params.yaml" />
-  <xacro:property name="params" value="${xacro.load_yaml(config_file)}"/>
-  <xacro:property name="wheel_radius" value="${params['/**']['ros__parameters']['wheel_radius']}"/>
-  <xacro:property name="track_width" value="${params['/**']['ros__parameters']['track_width']}"/>
-  <xacro:property name="collision_radius" value="${params['/**']['ros__parameters']['collision_radius']}"/>
-  <link name="base_footprint"/>
+  <xacro:property name="params" value="${xacro.load_yaml(config_file)}" />
+  <xacro:property name="wheel_radius" value="${params['/**']['ros__parameters']['wheel_radius']}" />
+  <xacro:property name="track_width" value="${params['/**']['ros__parameters']['track_width']}" />
+  <xacro:property name="collision_radius"
+    value="${params['/**']['ros__parameters']['collision_radius']}" />
+  <link name="base_footprint" />
   <joint name="base_joint" type="fixed">
-    <parent link="base_footprint"/>
-    <child link="base_link"/>
-    <origin xyz="0.0 0.0 0.010" rpy="0 0 0"/>
+    <parent link="base_footprint" />
+    <child link="base_link" />
+    <origin xyz="0.0 0.0 0.010" rpy="0 0 0" />
   </joint>
   <link name="base_link">
     <visual>
-      <origin xyz="-0.032 0 0.0" rpy="0 0 0"/>
+      <origin xyz="-0.032 0 0.0" rpy="0 0 0" />
       <geometry>
-        <mesh filename="package://nuturtle_description/meshes/burger_base.stl" scale="0.001 0.001 0.001"/>
+        <mesh filename="package://nuturtle_description/meshes/burger_base.stl"
+          scale="0.001 0.001 0.001" />
       </geometry>
-      <material name="$(arg color)"/>
+      <material name="$(arg color)" />
     </visual>
     <collision>
-      <origin xyz="-0.032 0 0.070" rpy="0 0 0"/>
+      <origin xyz="-0.032 0 0.070" rpy="0 0 0" />
       <geometry>
         <xacro:if value="${collision_radius &lt; 0}">
-          <box size="0.140 0.140 0.143"/>
+          <box size="0.140 0.140 0.143" />
         </xacro:if>
         <xacro:if value="${collision_radius &gt; 0}">
-          <cylinder radius="${collision_radius}" length="0.143"/>
+          <cylinder radius="${collision_radius}" length="0.143" />
         </xacro:if>
       </geometry>
     </collision>
     <inertial>
-      <origin xyz="0 0 0" rpy="0 0 0"/>
-      <mass value="8.2573504e-01"/>
-      <inertia ixx="2.2124416e-03" ixy="-1.2294101e-05" ixz="3.4938785e-05" iyy="2.1193702e-03" iyz="-5.0120904e-06" izz="2.0064271e-03" />
+      <origin xyz="0 0 0" rpy="0 0 0" />
+      <mass value="8.2573504e-01" />
+      <inertia ixx="2.2124416e-03" ixy="-1.2294101e-05" ixz="3.4938785e-05" iyy="2.1193702e-03"
+        iyz="-5.0120904e-06" izz="2.0064271e-03" />
     </inertial>
   </link>
   <joint name="wheel_left_joint" type="continuous">
-    <parent link="base_link"/>
-    <child link="wheel_left_link"/>
-    <origin xyz="0.0 ${track_width/2} 0.023" rpy="-1.57 0 0"/>
-    <axis xyz="0 0 1"/>
+    <parent link="base_link" />
+    <child link="wheel_left_link" />
+    <origin xyz="0.0 ${track_width/2} 0.023" rpy="-1.57 0 0" />
+    <axis xyz="0 0 1" />
   </joint>
   <link name="wheel_left_link">
     <visual>
-      <origin xyz="0 0 0" rpy="1.57 0 0"/>
+      <origin xyz="0 0 0" rpy="1.57 0 0" />
       <geometry>
-        <mesh filename="package://nuturtle_description/meshes/left_tire.stl" scale="0.001 0.001 0.001"/>
+        <mesh filename="package://nuturtle_description/meshes/left_tire.stl"
+          scale="0.001 0.001 0.001" />
       </geometry>
-      <material name="light_black"/>
+      <material name="light_black" />
     </visual>
     <collision>
-      <origin xyz="0 0 0" rpy="0 0 0"/>
+      <origin xyz="0 0 0" rpy="0 0 0" />
       <geometry>
-        <cylinder length="0.018" radius="${wheel_radius}"/>
+        <cylinder length="0.018" radius="${wheel_radius}" />
       </geometry>
     </collision>
@@ -63,25 +67,27 @@
       <origin xyz="0 0 0" />
       <mass value="2.8498940e-02" />
-      <inertia ixx="1.1175580e-05" ixy="-4.2369783e-11" ixz="-5.9381719e-09" iyy="1.1192413e-05" iyz="-1.4400107e-11" izz="2.0712558e-05" />
+      <inertia ixx="1.1175580e-05" ixy="-4.2369783e-11" ixz="-5.9381719e-09" iyy="1.1192413e-05"
+        iyz="-1.4400107e-11" izz="2.0712558e-05" />
     </inertial>
   </link>
   <joint name="wheel_right_joint" type="continuous">
-    <parent link="base_link"/>
-    <child link="wheel_right_link"/>
-    <origin xyz="0.0 -${track_width/2} 0.023" rpy="-1.57 0 0"/>
-    <axis xyz="0 0 1"/>
+    <parent link="base_link" />
+    <child link="wheel_right_link" />
+    <origin xyz="0.0 -${track_width/2} 0.023" rpy="-1.57 0 0" />
+    <axis xyz="0 0 1" />
   </joint>
   <link name="wheel_right_link">
     <visual>
-      <origin xyz="0 0 0" rpy="1.57 0 0"/>
+      <origin xyz="0 0 0" rpy="1.57 0 0" />
       <geometry>
-        <mesh filename="package://nuturtle_description/meshes/right_tire.stl" scale="0.001 0.001 0.001"/>
+        <mesh filename="package://nuturtle_description/meshes/right_tire.stl"
+          scale="0.001 0.001 0.001" />
       </geometry>
-      <material name="light_black"/>
+      <material name="light_black" />
     </visual>
     <collision>
-      <origin xyz="0 0 0" rpy="0 0 0"/>
+      <origin xyz="0 0 0" rpy="0 0 0" />
       <geometry>
-        <cylinder length="0.018" radius="${wheel_radius}"/>
+        <cylinder length="0.018" radius="${wheel_radius}" />
       </geometry>
     </collision>
@@ -89,17 +95,18 @@
       <origin xyz="0 0 0" />
       <mass value="2.8498940e-02" />
-      <inertia ixx="1.1175580e-05" ixy="-4.2369783e-11" ixz="-5.9381719e-09" iyy="1.1192413e-05" iyz="-1.4400107e-11" izz="2.0712558e-05" />
+      <inertia ixx="1.1175580e-05" ixy="-4.2369783e-11" ixz="-5.9381719e-09" iyy="1.1192413e-05"
+        iyz="-1.4400107e-11" izz="2.0712558e-05" />
     </inertial>
   </link>
   <joint name="caster_back_joint" type="fixed">
-    <parent link="base_link"/>
-    <child link="caster_back_link"/>
-    <origin xyz="-0.081 0 -0.004" rpy="-1.57 0 0"/>
+    <parent link="base_link" />
+    <child link="caster_back_link" />
+    <origin xyz="-0.081 0 -0.004" rpy="-1.57 0 0" />
   </joint>
   <link name="caster_back_link">
     <collision>
-      <origin xyz="0 0.001 0" rpy="0 0 0"/>
+      <origin xyz="0 0.001 0" rpy="0 0 0" />
       <geometry>
-        <box size="0.030 0.009 0.020"/>
+        <box size="0.030 0.009 0.020" />
       </geometry>
     </collision>
@@ -111,26 +118,26 @@
   </link>
   <joint name="imu_joint" type="fixed">
-    <parent link="base_link"/>
-    <child link="imu_link"/>
-    <origin xyz="-0.032 0 0.068" rpy="0 0 0"/>
+    <parent link="base_link" />
+    <child link="imu_link" />
+    <origin xyz="-0.032 0 0.068" rpy="0 0 0" />
   </joint>
-  <link name="imu_link"/>
+  <link name="imu_link" />
   <joint name="scan_joint" type="fixed">
-    <parent link="base_link"/>
-    <child link="base_scan"/>
-    <origin xyz="-0.032 0 0.172" rpy="0 0 0"/>
+    <parent link="base_link" />
+    <child link="base_scan" />
+    <origin xyz="-0.032 0 0.172" rpy="0 0 0" />
   </joint>
   <link name="base_scan">
     <visual>
-      <origin xyz="0 0 0.0" rpy="0 0 0"/>
+      <origin xyz="0 0 0.0" rpy="0 0 0" />
       <geometry>
-        <mesh filename="package://nuturtle_description/meshes/lds.stl" scale="0.001 0.001 0.001"/>
+        <mesh filename="package://nuturtle_description/meshes/lds.stl" scale="0.001 0.001 0.001" />
       </geometry>
-      <material name="light_black"/>
+      <material name="light_black" />
     </visual>
     <collision>
-      <origin xyz="0.015 0 -0.0065" rpy="0 0 0"/>
+      <origin xyz="0.015 0 -0.0065" rpy="0 0 0" />
       <geometry>
-        <cylinder length="0.0315" radius="0.055"/>
+        <cylinder length="0.0315" radius="0.055" />
       </geometry>
     </collision>

File: nuturtle_description/urdf/utils.xacro (robot description, xacro)
@@ -1,22 +1,22 @@
 <?xml version="1.0"?>
 <robot xmlns:xacro="https://www.ros.org/wiki/xacro" name="nuturtle_burger">
- <!-- Define some colors -->
+  <!-- Define some colors -->
   <material name="black">
-    <color rgba="0.0 0.0 0.0 1.0"/>
+    <color rgba="0.0 0.0 0.0 1.0" />
   </material>
   <material name="light_black">
-    <color rgba="0.4 0.4 0.4 1.0"/>
+    <color rgba="0.4 0.4 0.4 1.0" />
   </material>
   <material name="purple">
-    <color rgba="0.3 0.16 0.52 1.0"/>
+    <color rgba="0.3 0.16 0.52 1.0" />
   </material>
   <material name="green">
-    <color rgba="0.0 0.8 0.0 1.0"/>
+    <color rgba="0.0 0.8 0.0 1.0" />
   </material>
   <material name="blue">
-    <color rgba="0.0 0.0 0.8 1.0"/>
+    <color rgba="0.0 0.0 0.8 1.0" />
   </material>
   <material name="red">
-    <color rgba="0.8 0.0 0.0 1.0"/>
+    <color rgba="0.8 0.0 0.0 1.0" />
   </material>
 </robot>
